File: PCB/Arduino rx PLC/arduino rx.brd (EAGLE design)
At the start: 160 x 100 mm, 35 parts, among them J1 1X2-3.5MM, J2 1X5, J3 1X5, J4 1X2-3.5MM, J5 1X2-3.5MM, J6 1X2-3.5MM, T1 BC547, T2 BC547, T3 BC547, U1 ATMEGA328P_PDIP_EZ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

Commit message: final
Parts:
- removed J3: 1X5, adafruit:1X05-3.5MM
- added JP1, JP2: (no value), adafruit:1X06
- J1, J4, J5, J6: value 1X2-3.5MM -> (none); device adafruit:1X2-3.5MM -> SparkFun-Connectors:SCREWTERMINAL-3.5MM-2
- J2: value 1X5 -> (none); device adafruit:1X05-3.5MM -> SparkFun-Connectors:SCREWTERMINAL-3.5MM-2
- U1: value ATMEGA328P_PDIP_EZ -> 328P; device SparkFun-IC-Microcontroller:DIP28-SIMON-KIT -> SparkFun-IC-Microcontroller:DIP28
- moved 3 227.9 mm to (35.6, 59.7), turned to 270 degrees
- moved POWERLED3 224.9 mm to (41.9, 59.7), turned to 270 degrees
- moved 2 222.8 mm to (47.0, 59.7), turned to 270 degrees
- moved POWERLED2 220.4 mm to (53.3, 59.7), turned to 270 degrees
- moved 1 218.8 mm to (58.4, 59.7), turned to 270 degrees
- moved POWERLED1 217.0 mm to (64.8, 59.7), turned to 270 degrees
- moved J6 201.1 mm to (115.6, 27.9), turned to 90 degrees
- moved J5 189.2 mm to (115.6, 36.8), turned to 90 degrees
- moved J4 179.5 mm to (115.6, 45.7), turned to 90 degrees
- moved C3 173.8 mm to (21.6, 49.5)
- moved C4 173.8 mm to (21.6, 43.2)
- moved T3 168.8 mm to (80.0, 14.0), turned to 90 degrees
- moved T2 163.3 mm to (80.0, 36.8), turned to 90 degrees
- moved U$3 163.2 mm to (94.0, 15.2)
- moved U$2 158.6 mm to (94.0, 38.1)
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Connections:
- removed net N$11: J5.2, U$2.SWCOMMON
- removed net N$14: J6.1, U$3.SWCLOSED
- removed net N$15: J4.2, U$1.SWCOMMON
- new net NEUTRAL: J2.1, J4.2, J5.2, J6.2
- new net PHASE: J2.2, U$1.SWCOMMON, U$2.SWCOMMON, U$3.SWCOMMON
- net 12V: now also JP2.1; no longer J3.1
- net 5V: now also JP1.1, JP2.2; no longer J2.1, J3.2
- net GND: now also JP1.5, JP2.5; no longer J2.5, J3.5
- net N$10: now also J6.1, U$3.SWOPEN; no longer J6.2, U$3.SWCOMMON
- net N$8: now also U$2.SWOPEN; no longer U$2.SWCLOSED
- net N$9: now also U$1.SWOPEN; no longer U$1.SWCLOSED
- net RESET: now also JP1.2; no longer J2.2
- net RX: now also JP1.3; no longer J2.3
- net RX_PLC: now also JP2.3; no longer J3.3
- net TX: now also JP1.4; no longer J2.4
- net TX_PLC: now also JP2.4; no longer J3.4
Routing:
- net 5V: track 0.00 -> 521.0 mm, vias 0 -> 2
- net GND: track 0.00 -> 354.5 mm
- net RELAY1: track 0.00 -> 119.4 mm
- net PHASE: track 0.00 -> 103.5 mm
- net N$3: track 0.00 -> 70.1 mm
- net 12V: track 0.00 -> 60.8 mm
- net NEUTRAL: track 0.00 -> 54.7 mm
- net RELAY3: track 0.00 -> 42.0 mm
- net RESET: track 0.00 -> 39.9 mm
- net TX_PLC: track 0.00 -> 36.8 mm
- net RX_PLC: track 0.00 -> 33.7 mm
- net N$9: track 0.00 -> 31.6 mm
- net N$5: track 0.00 -> 29.8 mm
- net RELAY2: track 0.00 -> 25.0 mm
- net N$13: track 0.00 -> 24.9 mm
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Other:
- board size 160 x 100 mm -> 124.4 x 70.8 mm
- board text added: "PLC_RX"
