File: PCB/Arduino rx PLC/arduino rx.sch (EAGLE design)
At the start: 35 parts, among them J1 1X2-3.5MM, J2 1X5, J3 1X5, J4 1X2-3.5MM, J5 1X2-3.5MM, J6 1X2-3.5MM, T1 BC547, T2 BC547, T3 BC547, U1 ATMEGA328P_PDIP_EZ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

Commit message: final
Parts:
- removed J3: 1X5, adafruit:1X5
- added JP1, JP2: (no value), adafruit:PINHD-1X6
- J1, J4, J5, J6: value 1X2-3.5MM -> (none); device adafruit:1X2-3.5MM -> SparkFun-Connectors:CONN_023.5MM
- J2: value 1X5 -> (none); device adafruit:1X5 -> SparkFun-Connectors:CONN_023.5MM
- U1: value ATMEGA328P_PDIP_EZ -> 328P; device SparkFun-IC-Microcontroller:ATMEGA328P_PDIP_EZ -> SparkFun-IC-Microcontroller:ATMEGA328P_PDIP
Connections:
- removed net N$11: J5.2, U$2.SWCOMMON
- removed net N$14: J6.1, U$3.SWCLOSE
- removed net N$15: J4.2, U$1.SWCOMMON
- new net NEUTRAL: J2.1, J4.2, J5.2, J6.2
- new net PHASE: J2.2, U$1.SWCOMMON, U$2.SWCOMMON, U$3.SWCOMMON
- net 12V: now also JP2.1; no longer J3.1
- net 5V: now also JP1.1, JP2.2; no longer J2.1, J3.2
- net GND: now also JP1.5, JP2.5; no longer J2.5, J3.5
- net N$10: now also J6.1, U$3.SWOPEN; no longer J6.2, U$3.SWCOMMON
- net N$8: now also U$2.SWOPEN; no longer U$2.SWCLOSE
- net N$9: now also U$1.SWOPEN; no longer U$1.SWCLOSE
- net RESET: now also JP1.2; no longer J2.2
- net RX: now also JP1.3; no longer J2.3
- net RX_PLC: now also JP2.3; no longer J3.3
- net TX: now also JP1.4; no longer J2.4
- net TX_PLC: now also JP2.4; no longer J3.4
