File: PCB/Arduino tx PLC/arduino tx.sch (EAGLE design)
At the start: 20 parts, among them J1 1X2-3.5MM, J2 1X5, J3 1X5, U1 ATMEGA328P_PDIP_EZ, Y1 16MHz

Commit message: final
Parts:
- removed J2, J3: 1X5, adafruit:1X5
- added IC2: (no value), Lolin:NODEMCU_LOLINV3
- added SV1, SV2: (no value), con-lstb:MA05-1
- J1: value 1X2-3.5MM -> (none); device adafruit:1X2-3.5MM -> SparkFun-Connectors:CONN_025MM
- U1: value ATMEGA328P_PDIP_EZ -> 328P; device SparkFun-IC-Microcontroller:ATMEGA328P_PDIP_EZ -> SparkFun-IC-Microcontroller:ATMEGA328P_PDIP
- renumbered POWERLED3 to STATSLED
Connections:
- removed net LED3: 3.2, U1.PC2(ADC2)
- new net N$5: J1.1
- new net RX_DEV: IC2.D7, U1.PB1(OC1A)
- new net STATUSLED: 3.2, IC2.D0
- new net TX_DEV: IC2.D8, U1.PB2(SS/OC1B)
- net 12V: now also SV1.1; no longer J3.1
- net 5V: now also IC2.VIN, SV1.2, SV2.1; no longer J2.1, J3.2
- net GND: now also IC2.GND, SV1.5, SV2.5; no longer J1.1, J2.5, J3.5
- net RESET: now also SV2.2; no longer J2.2
- net RX: now also SV2.3; no longer J2.3
- net RX_PLC: now also SV1.3, U1.PB3(MOSI/OC2); no longer J3.3, U1.PD3(INT1)
- net TX: now also SV2.4; no longer J2.4
- net TX_PLC: now also SV1.4, U1.PB4(MISO); no longer J3.4, U1.PD4(XCK/T0)
